File: afterglow_nano/afterglow_nano.kicad_pcb (KiCad board)
At the start: 2 copper layers, 176.5 x 80 mm, 70 parts, among them J134 INPUT J133_IN_R, J134 OUTPUT J133_OUT_R, J138 INPUT J137_IN_C, J138 OUTPUT J137_OUT_C, Q1 2N3904, Q10 FQP27P06, Q11 FQP27P06, Q12 FQP27P06, Q13 FQP27P06, Q14 FQP27P06, Q15 FQP27P06, Q16 FQP27P06, Q17 FQP30N06L, Q18 FQP30N06L, Q19 FQP30N06L, Q2 2N3904, Q20 FQP30N06L, Q21 FQP30N06L, Q22 FQP30N06L, Q23 FQP30N06L, Q24 FQP30N06L, Q3 2N3904, Q4 2N3904, Q5 2N3904, Q6 2N3904, Q7 2N3904, Q8 2N3904, Q9 FQP27P06, U1 74LS165, U2 74LS165, U3 5V_Regulator, U4 arduino nano, U5 74HC595, U6 74HC595

Commit message: v1.1 progress
Parts:
- removed + 18V -: Conn_Power, Connectors_Molex:Molex_KK-41791-02_02x3.96mm_Straight
- removed J134 INPUT: J133_IN_R, Connectors_Molex:Molex_KK-6410-09_09x2.54mm_Straight
- removed J134 OUTPUT: J133_OUT_R, Connectors_Molex:Molex_KK-6410-09_09x2.54mm_Straight
- removed J138 INPUT: J137_IN_C, Connectors_Molex:Molex_KK-41791-9_9x3.96mm_Straight
- removed J138 OUTPUT: J137_OUT_C, Connectors_Molex:Molex_KK-41791-9_9x3.96mm_Straight
- removed the REF** at (49.0, 124.0)
- removed the REF** at (49.0, 56.0)
- removed the REF** at (215.5, 125.0)
- removed the REF** at (215.5, 55.0)
- added C4: 1000uF, Capacitors_THT:CP_Radial_D10.0mm_P5.00mm, F.Cu at (102.0, 122.0)
- added D2: 1N4004, Diodes_THT:D_5W_P10.16mm_Horizontal, F.Cu at (124.0, 122.0)
- added J3: Conn_Power, Connectors_Molex:Molex_KK-41791-02_02x3.96mm_Straight, F.Cu at (60.0, 124.0)
- added J34 INPUT: J133_IN_R, Connectors_Molex:Molex_KK-6410-09_09x2.54mm_Straight, F.Cu at (208.0, 60.9)
- added J38 INPUT: J137_IN_C, Connectors_Molex:Molex_KK-41791-9_9x3.96mm_Straight, F.Cu at (208.0, 87.0)
- added J4: J137_OUT_C, Connectors_Molex:Molex_KK-41791-9_9x3.96mm_Straight, F.Cu at (60.0, 113.8)
- added J5: J133_OUT_R, Connectors_Molex:Molex_KK-6410-09_09x2.54mm_Straight, F.Cu at (60.0, 75.3)
- added J6: J134_OUT_R, Connectors_Molex:Molex_KK-6410-09_09x2.54mm_Straight, F.Cu at (25.9, 75.2)
- added J7: J138_OUT_C, Connectors_Molex:Molex_KK-41791-9_9x3.96mm_Straight, F.Cu at (44.6, 113.8)
- added J8: J135_OUT_R, Connectors_Molex:Molex_KK-6410-09_09x2.54mm_Straight, F.Cu at (14.7, 75.7)
- added J9: 136_OUT_C, Connectors_Molex:Molex_KK-41791-03_03x3.96mm_Straight, F.Cu at (18.3, 90.9)
- added R18: 10k, Resistors_SMD:R_0805_HandSoldering, F.Cu at (146.5, 82.5)
- added R21: 220, Resistors_SMD:R_0805_HandSoldering, F.Cu at (76.5, 71.5)
- added R22: 220, Resistors_SMD:R_0805_HandSoldering, F.Cu at (88.0, 71.5)
- added R23: 220, Resistors_SMD:R_0805_HandSoldering, F.Cu at (99.5, 71.5)
- added R24: 220, Resistors_SMD:R_0805_HandSoldering, F.Cu at (111.5, 71.5)
- added R25: 220, Resistors_SMD:R_0805_HandSoldering, F.Cu at (77.0, 57.5)
- added R26: 220, Resistors_SMD:R_0805_HandSoldering, F.Cu at (88.5, 57.5)
- added R27: 220, Resistors_SMD:R_0805_HandSoldering, F.Cu at (99.8, 57.5)
- added R28: 220, Resistors_SMD:R_0805_HandSoldering, F.Cu at (111.0, 57.5)
- added REF**: MountingHole_4.3mm_M4_DIN965, Mounting_Holes:MountingHole_4.3mm_M4_DIN965, F.Cu at (213.5, 55.0)
- RN3: value 10k -> 2k
- moved D1 72.7 mm to (187.7, 68.0), turned to 0 degrees
- moved R9 57.3 mm to (172.0, 72.5), turned to 180 degrees
- moved C3 27.0 mm to (149.0, 122.0), turned to 0 degrees
- moved C2 23.0 mm to (155.0, 122.0), turned to 180 degrees
- moved U3 22.1 mm to (131.0, 122.0)
- moved C1 17.0 mm to (143.0, 122.0), turned to 0 degrees
- moved afterglow 11.0 mm to (36.5, 99.0)
- moved FLAKIE 3.00 mm to (183.5, 58.0)
- moved CONFIG 2.09 mm to (171.2, 59.4)
- moved F1 0.50 mm to (93.5, 122.0)
Connections:
- C1 pad 1: /18V -> Net-(C1-Pad1)
- Q17 pad 1: /RO1 -> Net-(Q17-Pad1)
- Q18 pad 1: /RO2 -> Net-(Q18-Pad1)
- Q19 pad 1: /RO3 -> Net-(Q19-Pad1)
- Q20 pad 1: /RO4 -> Net-(Q20-Pad1)
- Q21 pad 1: /RO5 -> Net-(Q21-Pad1)
- Q22 pad 1: /RO6 -> Net-(Q22-Pad1)
- Q23 pad 1: /RO7 -> Net-(Q23-Pad1)
- Q24 pad 1: /RO8 -> Net-(Q24-Pad1)
- R9 pad 1: Net-(R9-Pad1) -> Net-(D1-Pad2)
- R9 pad 2: Net-(D1-Pad2) -> Net-(R9-Pad2)
- U3 pad 1: /18V -> Net-(C1-Pad1)
- U4 pad 11: Net-(U4-Pad11) -> Net-(R9-Pad2)
- U4 pad 20: Net-(U4-Pad20) -> Net-(R18-Pad2)
- U4 pad 26: Net-(R9-Pad1) -> Net-(U4-Pad26)
- U5 pad 13: GND -> Net-(R18-Pad2)
- U6 pad 13: GND -> Net-(R18-Pad2)
Routing:
- net Net-(R18-Pad2): track 0.00 -> 102.6 mm, vias 0 -> 2
- net Net-(C1-Pad1): track 0.00 -> 47.1 mm
- net VCC: track 325.5 -> 284.2 mm
- net Net-(R9-Pad1): track 41.1 -> 0.00 mm, vias 1 -> 0
- net /18V: track 186.7 -> 166.7 mm, vias 1 -> 0
- net GND: track 674.6 -> 692.1 mm, vias 2 -> 1
- net /OUT_CLK: track 112.6 -> 97.4 mm
- net Net-(D1-Pad2): track 4.08 -> 17.5 mm
- net /RO6: track 81.7 -> 73.8 mm
- net /RO8: track 43.9 -> 36.0 mm
- net /RO5: track 99.9 -> 92.1 mm
- net /RO7: track 63.6 -> 55.8 mm
- net Net-(R9-Pad2): track 0.00 -> 7.52 mm
- net Net-(Q22-Pad1): track 0.00 -> 7.20 mm
- net Net-(Q24-Pad1): track 0.00 -> 7.18 mm
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Other:
- board size 176.5 x 80 mm -> 185 x 80 mm
- board text added: "v1.1"
- board text removed: "v1.0"

Commit message: v1.1 PCB
Parts:
- added ?: MountingHole_4.3mm_M4_DIN965, Mounting_Holes:MountingHole_4.3mm_M4_DIN965, F.Cu at (30.5, 55.5)
- added ?: MountingHole_4.3mm_M4_DIN965, Mounting_Holes:MountingHole_4.3mm_M4_DIN965, F.Cu at (30.5, 124.5)
- added ?: MountingHole_4.3mm_M4_DIN965, Mounting_Holes:MountingHole_4.3mm_M4_DIN965, F.Cu at (212.5, 124.5)
- + 18V -: renamed from J3
- J133 OUT: renamed from J5
- J134 OUT: renamed from J6
- J135 OUT: renamed from J8
- J136 OUT: renamed from J9
- J137 OUT: renamed from J4
- J138 OUT: renamed from J7
- J34 IN: renamed from J34 INPUT
- J38 IN: renamed from J38 INPUT
- moved J136 OUT 42.7 mm to (42.0, 126.4)
- moved J135 OUT 23.3 mm to (38.0, 75.3)
- moved J134 OUT 23.1 mm to (49.0, 75.3)
- moved afterglow 18.3 mm to (29.0, 115.7)
- moved J138 OUT 2.60 mm to (42.0, 113.8)
- moved ? 0.71 mm to (213.0, 55.5)
- renumbered REF** to ?
Routing:
- net /J137_CO7: track 53.0 -> 119.1 mm
- net /J137_CO8: track 63.2 -> 127.4 mm
- net /J133_RO1: track 69.4 -> 93.4 mm
- net /J133_RO7: track 68.4 -> 90.4 mm
- net /J133_RO5: track 68.6 -> 90.6 mm
- net /J133_RO4: track 71.8 -> 93.8 mm
- net /J133_RO8: track 68.9 -> 90.9 mm
- net /J133_RO6: track 66.9 -> 88.9 mm
- net /J133_RO2: track 69.1 -> 91.1 mm
- net /J133_RO3: track 72.2 -> 94.2 mm
- net /J137_CO6: track 49.1 -> 67.1 mm
- net /J137_CO2: track 45.9 -> 63.9 mm
- net /J137_CO4: track 75.9 -> 93.9 mm
- net /J137_CO3: track 60.5 -> 78.5 mm
- net /J137_CO1: track 37.7 -> 55.7 mm
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Other:
- board size 185 x 80 mm -> 193.5 x 80 mm

Commit message: Minor trace fix
Routing:
- net /J137_CO8: track 127.4 -> 125.8 mm
- net /J137_CO7: track 119.1 -> 117.5 mm
Changed lines of the file:
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@@
 (kicad_pcb (version 4) (host pcbnew 4.0.7)
   (general
-    (links 0)
-    (no_connects 26)
+    (links 240)
+    (no_connects 4)
     (area 17.571429 49.475 225.928572 130.625)
     (thickness 1.6)
     (drawings 31)
-    (tracks 1136)
+    (tracks 1135)
     (zones 0)
     (modules 85)
@@
   (segment (start 177.25 76.75) (end 178.5 75.5) (width 0.5) (layer F.Cu) (net 23))
   (segment (start 196.84 81.32) (end 196.8 81.28) (width 0.5) (layer F.Cu) (net 23))
+  (segment (start 60.603478 113.7744) (end 66.652879 107.724999) (width 1.75) (layer B.Cu) (net 24))
+  (segment (start 60 113.7744) (end 60.603478 113.7744) (width 1.75) (layer B.Cu) (net 24))
   (segment (start 42 113.7792) (end 59.9958 113.7792) (width 1.75) (layer B.Cu) (net 24))
   (segment (start 59.9958 113.7792) (end 60 113.775) (width 1.75) (layer B.Cu) (net 24))
   (segment (start 76.54 110) (end 88.38 98.16) (width 0.5) (layer F.Cu) (net 24))
   (segment (start 88.38 98.16) (end 88.38 98) (width 0.5) (layer F.Cu) (net 24))
-  (segment (start 60 113.7744) (end 60.603478 113.7744) (width 1.75) (layer B.Cu) (net 24))
   (segment (start 66.652879 107.724999) (end 75.621999 107.724999) (width 1.75) (layer B.Cu) (net 24))
-  (segment (start 60.603478 113.7744) (end 66.652879 107.724999) (width 1.75) (layer B.Cu) (net 24))
   (segment (start 76.54 108.727208) (end 76.54 110) (width 1.75) (layer B.Cu) (net 24))
   (segment (start 75.621999 107.724999) (end 76.54 108.643) (width 1.75) (layer B.Cu) (net 24))
   (segment (start 76.54 108.643) (end 76.54 108.727208) (width 1.75) (layer B.Cu) (net 24))
+  (segment (start 60.603478 109.812) (end 64.940489 105.474989) (width 1.75) (layer B.Cu) (net 25))
   (segment (start 60 109.8126) (end 42.0042 109.8126) (width 1.75) (layer B.Cu) (net 25))
   (segment (start 42.0042 109.8126) (end 42 109.8168) (width 1.75) (layer B.Cu) (net 25))
@@
   (segment (start 88 100.92) (end 90.92 98) (width 0.5) (layer F.Cu) (net 25))
   (segment (start 60 109.812) (end 60.603478 109.812) (width 1.75) (layer B.Cu) (net 25))
-  (segment (start 60.603478 109.812) (end 64.940489 105.474989) (width 1.75) (layer B.Cu) (net 25))
   (segment (start 64.940489 105.474989) (end 85.209991 105.474989) (width 1.75) (layer B.Cu) (net 25))
   (segment (start 85.209991 105.474989) (end 88 108.264998) (width 1.75) (layer B.Cu) (net 25))
@@
   (segment (start 85.209991 87.474989) (end 88 90.264998) (width 1.75) (layer B.Cu) (net 29))
   (segment (start 88 90.264998) (end 88 90.727208) (width 1.75) (layer B.Cu) (net 29))
+  (segment (start 60 90.0006) (end 60 90) (width 1.75) (layer F.Cu) (net 30))
   (segment (start 53.5 113.931994) (end 53.5 111.5) (width 1.75) (layer F.Cu) (net 30))
   (segment (start 53.5 111.5) (end 53.5 92.7506) (width 1.75) (layer F.Cu) (net 30))
@@
   (segment (start 99.46 92) (end 99.46 93.84) (width 0.5) (layer F.Cu) (net 30))
   (segment (start 99.46 93.84) (end 103.62 98) (width 0.5) (layer F.Cu) (net 30))
-  (segment (start 60 90) (end 61.08739 88.91261) (width 1.75) (layer B.Cu) (net 30))
   (segment (start 61.08739 88.91261) (end 66.398202 88.91261) (width 1.75) (layer B.Cu) (net 30))
   (segment (start 99.46 90.727208) (end 99.46 92) (width 1.75) (layer B.Cu) (net 30))
@@
   (segment (start 60 82.0752) (end 60.249924 82.0752) (width 1.75) (layer B.Cu) (net 32))
   (segment (start 61.399693 83.224969) (end 103.049971 83.224969) (width 1.75) (layer B.Cu) (net 32))
-  (segment (start 60.249924 82.0752) (end 61.399693 83.224969) (width 1.75) (layer B.Cu) (net 32))
   (segment (start 103.049971 83.224969) (end 110.54 90.714998) (width 1.75) (layer B.Cu) (net 32))
   (segment (start 110.54 90.714998) (end 110.54 90.727208) (width 1.75) (layer B.Cu) (net 32))
