File: afterglow_nano_smd/afterglow_nano_smd.kicad_pcb (KiCad board)
At the start: 2 copper layers, 116.5 x 81 mm, 114 parts, among them J1 J137_IN_C, J2 J133_IN_R, J3 Conn_Power, J4 J133_OUT_R, J5 J137_OUT_C, J6 J134_OUT_R, J7 J138_OUT_C, J8 J135_OUT_R, J9 136_OUT_C, Q1 IRF5305, Q10 IRL2905, Q11 IRL2905, Q12 IRL2905, Q13 IRL2905, Q14 IRL2905, Q15 IRL2905, Q16 IRL2905, Q2 IRF5305, Q3 IRF5305, Q4 IRF5305, Q5 IRF5305, Q6 IRF5305, Q7 IRF5305, Q8 IRF5305, Q9 IRL2905, U1 74LS165, U2 74LS165, U3 5V_Regulator, U5 74HC595, U6 74HC595, U7 ULN2803A

Commit message: PCB complete
Parts:
- + 18V -: renamed from J3
- Arduino Nano: renamed from A1
- J133 OUT: renamed from J4
- J134 IN: renamed from J2
- J134 OUT: renamed from J6
- J135 OUT: renamed from J8
- J136 OUT: renamed from J9
- J137 OUT: renamed from J5
- J138 IN: renamed from J1
- J138 OUT: renamed from J7
Other:
- board text removed: "(c) 2017 morbid cornflakes"
- board text removed: "v1.2"
