File: afterglow_nano_smd/afterglow_nano_smd.kicad_pcb (KiCad board)
At the start: 2 copper layers, 116.5 x 81 mm, 114 parts, among them J133 OUT J133_OUT_R, J134 IN J133_IN_R, J134 OUT J134_OUT_R, J135 OUT J135_OUT_R, J136 OUT 136_OUT_C, J137 OUT J137_OUT_C, J138 IN J137_IN_C, J138 OUT J138_OUT_C, Q1 IRF5305, Q10 IRL2905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

Commit message: Added the configuration DIP switch back - it might be handy after all
Parts:
- removed TEST: Jumper, Pin_Headers:Pin_Header_Straight_1x02_Pitch2.54mm
- added SW1: CFG, Buttons_Switches_THT:SW_DIP_x4_W7.62mm_Slide, F.Cu at (118.0, 64.0)
- A1: renamed from Arduino Nano
- J1: renamed from J138 IN
- J2: renamed from J134 IN
- J3: renamed from + 18V -
- J4: renamed from J133 OUT
- J5: renamed from J137 OUT
- J6: renamed from J134 OUT
- J7: renamed from J138 OUT
- J8: renamed from J135 OUT
- J9: renamed from J136 OUT
- moved FLAKIE 18.4 mm to (102.5, 72.5)
- renumbered GND to TP1, 5V to TP2, 18V to TP3
Connections:
- A1 pad 1: Net-(A1-Pad1) -> (no net)
- A1 pad 15: Net-(A1-Pad15) -> (no net)
- A1 pad 16: Net-(A1-Pad16) -> (no net)
- A1 pad 17: Net-(A1-Pad17) -> (no net)
- A1 pad 18: Net-(A1-Pad18) -> (no net)
- A1 pad 2: Net-(A1-Pad2) -> (no net)
- A1 pad 21: Net-(A1-Pad21) -> (no net)
- A1 pad 22: Net-(A1-Pad22) -> (no net)
- A1 pad 23: Net-(A1-Pad23) -> (no net)
- A1 pad 24: Net-(A1-Pad24) -> (no net)
- A1 pad 25: Net-(A1-Pad25) -> (no net)
- A1 pad 26: Net-(A1-Pad26) -> (no net)
- A1 pad 28: Net-(A1-Pad28) -> (no net)
- A1 pad 3: Net-(A1-Pad3) -> (no net)
- A1 pad 30: Net-(A1-Pad30) -> (no net)
- J1 pad 8: Net-(J1-Pad8) -> (no net)
- J2 pad 3: Net-(J2-Pad3) -> (no net)
- J4 pad 3: Net-(J4-Pad3) -> (no net)
- J5 pad 8: Net-(J5-Pad8) -> (no net)
- J6 pad 3: Net-(J6-Pad3) -> (no net)
- J7 pad 8: Net-(J7-Pad8) -> (no net)
- J8 pad 3: Net-(J8-Pad3) -> (no net)
- J9 pad 1: Net-(J9-Pad1) -> (no net)
- U1 pad 7: Net-(U1-Pad7) -> (no net)
- U2 pad 10: Net-(U2-Pad10) -> (no net)
- U2 pad 7: Net-(U2-Pad7) -> (no net)
- U6 pad 9: Net-(U6-Pad9) -> (no net)
Routing:
- net Net-(A1-Pad12): track 0.00 -> 39.3 mm, vias 0 -> 1
- net Net-(A1-Pad14): track 0.00 -> 37.8 mm
- net Net-(A1-Pad11): track 0.00 -> 37.0 mm, vias 0 -> 1
- net GND: track 315.2 -> 334.4 mm
- net Net-(A1-Pad13): track 19.3 -> 38.0 mm
- net /J133_RO7: track 39.6 -> 36.6 mm
- net /IN_CLK: track 64.4 -> 63.6 mm

Commit message: PCB v1.3 ready
Parts:
- + 18V -: renamed from J3
- Arduino Nano: renamed from A1
- renumbered TP3 to 18V, TP2 to 5V, SW1 to CFG, TP1 to GND
Other:
- board text added: "4"
- board text added: "J133 OUT"
- board text added: "J134 OUT"
- board text added: "J135 IN"
- board text added: "J135 OUT"
- board text added: "J136 OUT"
- board text added: "J137 OUT"
- board text added: "J138 IN"
- board text added: "J138 OUT"
Changed lines of the file:
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@@
   (general
     (thickness 1.6)
-    (drawings 41)
+    (drawings 57)
     (tracks 914)
     (zones 0)
@@
   (page A4)
   (title_block
-    (title "afterglow 1.1")
+    (title "afterglow 1.3")
     (company "morbid cornflakes")
   )
   (layers
-    (0 F.Cu signal)
-    (31 B.Cu signal)
+    (0 F.Cu signal hide)
+    (31 B.Cu signal hide)
     (32 B.Adhes user hide)
     (33 F.Adhes user hide)
-    (34 B.Paste user)
-    (35 F.Paste user)
+    (34 B.Paste user hide)
+    (35 F.Paste user hide)
     (36 B.SilkS user)
     (37 F.SilkS user)
-    (38 B.Mask user)
-    (39 F.Mask user)
-    (40 Dwgs.User user)
+    (38 B.Mask user hide)
+    (39 F.Mask user hide)
+    (40 Dwgs.User user hide)
     (41 Cmts.User user hide)
     (42 Eco1.User user hide)
@@
     (45 Margin user hide)
     (46 B.CrtYd user hide)
-    (47 F.CrtYd user)
+    (47 F.CrtYd user hide)
     (48 B.Fab user hide)
     (49 F.Fab user hide)
   )
   (setup
-    (last_trace_width 1.75)
+    (last_trace_width 0.5)
     (user_trace_width 0.25)
     (user_trace_width 0.5)
@@
     (descr "Through hole straight pin header, 1x01, 2.54mm pitch, single row")
     (tags "Through hole pin header THT 1x01 2.54mm single row")
-    (fp_text reference TP3 (at 1.5 4 180) (layer F.SilkS)
+    (fp_text reference 18V (at 1.5 4 180) (layer F.SilkS)
       (effects (font (size 1 1) (thickness 0.15)))
     )
@@
     (descr "Through hole straight pin header, 1x01, 2.54mm pitch, single row")
     (tags "Through hole pin header THT 1x01 2.54mm single row")
-    (fp_text reference TP2 (at 1 3.5 180) (layer F.SilkS)
+    (fp_text reference 5V (at 1 3.5 180) (layer F.SilkS)
       (effects (font (size 1 1) (thickness 0.15)))
     )
@@
     (descr "Through hole straight pin header, 1x01, 2.54mm pitch, single row")
     (tags "Through hole pin header THT 1x01 2.54mm single row")
-    (fp_text reference TP1 (at 0 4 180) (layer F.SilkS)
+    (fp_text reference GND (at 0 4 180) (layer F.SilkS)
       (effects (font (size 1 1) (thickness 0.15)))
     )
@@
     (descr "Arduino Nano, http://www.mouser.com/pdfdocs/Gravitech_Arduino_Nano3_0.pdf")
     (tags "Arduino Nano")
-    (fp_text reference A1 (at 7.5 18.5 270) (layer F.SilkS)
+    (fp_text reference "Arduino Nano" (at 7.5 18.5 270) (layer F.SilkS)
       (effects (font (size 1 1) (thickness 0.15)))
     )
@@
     (descr "Connector Headers with Friction Lock, 26-60-4020, http://www.molex.com/pdm_docs/sd/026604020_sd.pdf")
     (tags "connector molex kk_41791 26-60-4020")
-    (fp_text reference J7 (at 14.455 -6.35 90) (layer F.SilkS)
+    (fp_text reference J7 (at 34.5 -0.01 180) (layer F.SilkS)
       (effects (font (size 1 1) (thickness 0.15)))
     )
@@
     (descr "Connector Headers with Friction Lock, 26-60-4020, http://www.molex.com/pdm_docs/sd/026604020_sd.pdf")
     (tags "connector molex kk_41791 26-60-4020")
-    (fp_text reference J5 (at 14.5 -6.35 90) (layer F.SilkS)
+    (fp_text reference J5 (at 35 -0.25 180) (layer F.SilkS)
       (effects (font (size 1 1) (thickness 0.15)))
     )
@@
     (descr "Connector Headers with Friction Lock, 26-60-4020, http://www.molex.com/pdm_docs/sd/026604020_sd.pdf")
     (tags "connector molex kk_41791 26-60-4020")
-    (fp_text reference J1 (at 14.535 -6.455 270) (layer F.SilkS)
+    (fp_text reference J1 (at 34.535 -0.455) (layer F.SilkS)
       (effects (font (size 1 1) (thickness 0.15)))
     )
@@
     (descr "Connector Headers with Friction Lock, 22-27-2091, http://www.molex.com/pdm_docs/sd/022272021_sd.pdf")
     (tags "connector molex kk_6410 22-27-2091")
-    (fp_text reference J2 (at 10.435 -4.55 270) (layer F.SilkS)
+    (fp_text reference J2 (at -3.065 -0.05) (layer F.SilkS)
       (effects (font (size 1 1) (thickness 0.15)))
     )
@@
     (descr "Connector Headers with Friction Lock, 26-60-4020, http://www.molex.com/pdm_docs/sd/026604020_sd.pdf")
     (tags "connector molex kk_41791 26-60-4020")
-    (fp_text reference J3 (at 2.2 -6.75 90) (layer F.SilkS)
+    (fp_text reference "+ 18V -" (at 1.7 -6.75 90) (layer F.SilkS)
       (effects (font (size 1 1) (thickness 0.15)))
     )
@@
     (descr "Connector Headers with Friction Lock, 22-27-2091, http://www.molex.com/pdm_docs/sd/022272021_sd.pdf")
     (tags "connector molex kk_6410 22-27-2091")
-    (fp_text reference J6 (at 9.9 -4.36 90) (layer F.SilkS)
+    (fp_text reference J6 (at 22.9 0.14 180) (layer F.SilkS)
       (effects (font (size 1 1) (thickness 0.15)))
     )
@@
     (descr "Connector Headers with Friction Lock, 22-27-2091, http://www.molex.com/pdm_docs/sd/022272021_sd.pdf")
     (tags "connector molex kk_6410 22-27-2091")
-    (fp_text reference J8 (at 9.9 -4.7 90) (layer F.SilkS)
+    (fp_text reference J8 (at 22.9 -0.2 180) (layer F.SilkS)
       (effects (font (size 1 1) (thickness 0.15)))
     )
@@
     (descr "Connector Headers with Friction Lock, 26-60-4020, http://www.molex.com/pdm_docs/sd/026604020_sd.pdf")
     (tags "connector molex kk_41791 26-60-4020")
-    (fp_text reference J9 (at 4.445 -6.35 90) (layer F.SilkS)
+    (fp_text reference J9 (at -2.8 -0.51 180) (layer F.SilkS)
       (effects (font (size 1 1) (thickness 0.15)))
     )
@@
     (pad 2 thru_hole circle (at 5 0 180) (size 2 2) (drill 1) (layers *.Cu *.Mask)
       (net 2 GND))
-    (model ${KISYS3DMOD}/Capacitors_THT.3dshapes/CP_Radial_D10.0mm_P5.00mm.wrl
+    (model /usr/share/kicad/modules/Capacitor_THT.pretty/CP_Radial_D10.0mm_P5.00mm.kicad_mod
       (at (xyz 0 0 0))
       (scale (xyz 1 1 1))
@@
     (descr "Connector Headers with Friction Lock, 22-27-2091, http://www.molex.com/pdm_docs/sd/022272021_sd.pdf")
     (tags "connector molex kk_6410 22-27-2091")
-    (fp_text reference J4 (at 9.9 -4.52 90) (layer F.SilkS)
+    (fp_text reference J4 (at 22.9 -0.02 180) (layer F.SilkS)
       (effects (font (size 1 1) (thickness 0.15)))
     )
@@
     (descr "4x-dip-switch, Slide, row spacing 7.62 mm (300 mils)")
     (tags "DIP Switch Slide 7.62mm 300mil")
-    (fp_text reference SW1 (at 3.81 -3.48 180) (layer F.SilkS)
+    (fp_text reference CFG (at 4 11.5 180) (layer F.SilkS)
       (effects (font (size 1 1) (thickness 0.15)))
     )
@@
       (rotate (xyz 0 0 90))
     )
+    (model ${KISYS3DMOD}/Button_Switch_THT.3dshapes/SW_DIP_x4_W7.62mm_Slide.step
+      (at (xyz 0 0 0))
+      (scale (xyz 1 1 1))
+      (rotate (xyz 0 0 0))
+    )
+  )
+  (gr_text 4 (at 120.5 56.5) (layer F.SilkS)
+    (effects (font (size 1 1) (thickness 0.15)))
+  )
+  (gr_text 1 (at 120.5 64) (layer F.SilkS)
+    (effects (font (size 1 1) (thickness 0.15)))
+  )
+  (gr_text "J138 IN" (at 137.5 103 90) (layer F.SilkS)
+    (effects (font (size 1 1) (thickness 0.15)))
+  )
+  (gr_text "J135 IN" (at 137.5 72.5 90) (layer F.SilkS)
+    (effects (font (size 1 1) (thickness 0.15)))
+  )
+  (gr_text "J133 OUT" (at 54 65 90) (layer F.SilkS)
+    (effects (font (size 1 1) (thickness 0.15)))
+  )
+  (gr_text "J134 OUT" (at 43.5 65 90) (layer F.SilkS)
+    (effects (font (size 1 1) (thickness 0.15)))
+  )
+  (gr_text "J135 OUT" (at 33.5 65 90) (layer F.SilkS)
+    (effects (font (size 1 1) (thickness 0.15)))
+  )
+  (gr_line (start 53.303582 69.687208) (end 54.303582 70.187208) (layer F.SilkS) (width 0.2))
+  (gr_line (start 53.303582 70.687208) (end 53.303582 69.687208) (layer F.SilkS) (width 0.2))
+  (gr_line (start 54.303582 70.187208) (end 53.303582 70.687208) (layer F.SilkS) (width 0.2))
+  (gr_line (start 43.303582 70.687208) (end 43.303582 69.687208) (layer F.SilkS) (width 0.2))
+  (gr_line (start 43.303582 69.687208) (end 44.303582 70.187208) (layer F.SilkS) (width 0.2))
+  (gr_line (start 44.303582 70.187208) (end 43.303582 70.687208) (layer F.SilkS) (width 0.2))
+  (gr_text "J136 OUT" (at 35 121 90) (layer F.SilkS)
+    (effects (font (size 1 1) (thickness 0.15)))
+  )
+  (gr_text "J137 OUT" (at 50.5 98 90) (layer F.SilkS)
+    (effects (font (size 1 1) (thickness 0.15)))
+  )
+  (gr_text "J138 OUT" (at 35 98 90) (layer F.SilkS)
+    (effects (font (size 1 1) (thickness 0.15)))
   )
   (gr_line (start 50.603582 85.087208) (end 51.603582 85.587208) (layer F.SilkS) (width 0.2))
