File: afterglow_nano_smd/afterglow_nano_smd.sch (KiCad schematic (older format))
At the start: 116 parts, among them J1 J137_IN_C, J2 J133_IN_R, J3 Conn_Power, J4 J133_OUT_R, J5 J137_OUT_C, J6 J134_OUT_R, J7 J138_OUT_C, J8 J135_OUT_R, J9 136_OUT_C, Q1 IRFR9024, Q10 IRLR024, Q11 IRLR024, Q12 IRLR024, Q13 IRLR024, Q14 IRLR024, Q15 IRLR024, Q16 IRLR024, Q2 IRFR9024, Q3 IRFR9024, Q4 IRFR9024, Q5 IRFR9024, Q6 IRFR9024, Q7 IRFR9024, Q8 IRFR9024, Q9 IRLR024, SW1 CFG, U1 74LS165, U2 74LS165, U3 5V_Regulator, U5 74HC595, U6 74HC595, U7 ULN2803A

Commit message: The row pullups must be 1k instead of 10k. Other minor adjustments.
Parts:
- R10, R11, R12, R13, R14, R15, R16, R9: value 10k -> 1k
Changed lines of the file:
@@
 P 2800 5700
 F 0 "R9" V 2850 5500 50  0000 C CNN
-F 1 "10k" V 2800 5700 50  0000 C CNN
+F 1 "1k" V 2800 5700 50  0000 C CNN
 F 2 "Resistors_SMD:R_0805_HandSoldering" V 2730 5700 50  0001 C CNN
 F 3 "" H 2800 5700 50  0001 C CNN
@@
 P 2800 5800
 F 0 "R10" V 2850 5600 50  0000 C CNN
-F 1 "10k" V 2800 5800 50  0000 C CNN
+F 1 "1k" V 2800 5800 50  0000 C CNN
 F 2 "Resistors_SMD:R_0805_HandSoldering" V 2730 5800 50  0001 C CNN
 F 3 "" H 2800 5800 50  0001 C CNN
@@
 P 2800 5900
 F 0 "R11" V 2850 5700 50  0000 C CNN
-F 1 "10k" V 2800 5900 50  0000 C CNN
+F 1 "1k" V 2800 5900 50  0000 C CNN
 F 2 "Resistors_SMD:R_0805_HandSoldering" V 2730 5900 50  0001 C CNN
 F 3 "" H 2800 5900 50  0001 C CNN
@@
 P 2800 6000
 F 0 "R12" V 2850 5800 50  0000 C CNN
-F 1 "10k" V 2800 6000 50  0000 C CNN
+F 1 "1k" V 2800 6000 50  0000 C CNN
 F 2 "Resistors_SMD:R_0805_HandSoldering" V 2730 6000 50  0001 C CNN
 F 3 "" H 2800 6000 50  0001 C CNN
@@
 P 2800 6100
 F 0 "R13" V 2850 5900 50  0000 C CNN
-F 1 "10k" V 2800 6100 50  0000 C CNN
+F 1 "1k" V 2800 6100 50  0000 C CNN
 F 2 "Resistors_SMD:R_0805_HandSoldering" V 2730 6100 50  0001 C CNN
 F 3 "" H 2800 6100 50  0001 C CNN
@@
 P 2800 6200
 F 0 "R14" V 2850 6000 50  0000 C CNN
-F 1 "10k" V 2800 6200 50  0000 C CNN
+F 1 "1k" V 2800 6200 50  0000 C CNN
 F 2 "Resistors_SMD:R_0805_HandSoldering" V 2730 6200 50  0001 C CNN
 F 3 "" H 2800 6200 50  0001 C CNN
@@
 P 2800 6300
 F 0 "R15" V 2850 6100 50  0000 C CNN
-F 1 "10k" V 2800 6300 50  0000 C CNN
+F 1 "1k" V 2800 6300 50  0000 C CNN
 F 2 "Resistors_SMD:R_0805_HandSoldering" V 2730 6300 50  0001 C CNN
 F 3 "" H 2800 6300 50  0001 C CNN
@@
 P 2800 6400
 F 0 "R16" V 2850 6200 50  0000 C CNN
-F 1 "10k" V 2800 6400 50  0000 C CNN
+F 1 "1k" V 2800 6400 50  0000 C CNN
 F 2 "Resistors_SMD:R_0805_HandSoldering" V 2730 6400 50  0001 C CNN
 F 3 "" H 2800 6400 50  0001 C CNN
