File: afterglow_pcb_v14/afterglow_nano_smd.sch (KiCad schematic (older format))
At the start: 125 parts, among them J1 J137_IN_C, J2 J133_IN_R, J3 Conn_Power, J4 J133_OUT_R, J5 J137_OUT_C, J6 J134_OUT_R, J7 J138_OUT_C, J8 J135_OUT_R, J9 136_OUT_C, Q1 IRFR9024, Q10 IRLR024, Q11 IRLR024, Q12 IRLR024, Q13 IRLR024, Q14 IRLR024, Q15 IRLR024, Q16 IRLR024, Q2 IRFR9024, Q3 IRFR9024, Q4 IRFR9024, Q5 IRFR9024, Q6 IRFR9024, Q7 IRFR9024, Q8 IRFR9024, Q9 IRLR024, SW1 CFG, U1 74LS165, U2 74LS165, U3 5V_Regulator, U5 74HC595, U6 74HC595, U7 ULN2803A

Commit message: Some schematics update
Parts:
- A1: symbol afterglow_nano_smd-rescue:Arduino_Nano_v3.x-MCU_Module -> afterglow_nano_smd-rescue:Arduino_Nano_v3.x-MCU_Module-afterglow_nano_smd-rescue
Changed lines of the file:
@@
 	6200 9300 6200 9400
 $Comp
-L afterglow_nano_smd-rescue:Arduino_Nano_v3.x-MCU_Module A1
+L afterglow_nano_smd-rescue:Arduino_Nano_v3.x-MCU_Module-afterglow_nano_smd-rescue A1
 U 1 1 5B9C7C51
 P 8000 5350
