File: afterglow_stern_pcb_v10/afterglow_nano_smd.kicad_pcb (KiCad board)
At the start: 2 copper layers, 128.7 x 81 mm, 118 parts, among them J1 J13_IN_C, J2 J12_IN_R, J3 J12_OUT_R, J5 J13_OUT_C, Q1 FQP11P06, Q10 FQP13N06L, Q11 FQP13N06L, Q12 FQP13N06L, Q13 FQP13N06L, Q14 FQP13N06L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

Commit message: Kicad 6
Parts:
- added REF**: MountingHole_5mm_Pad, Mounting_Holes:MountingHole_5mm_Pad, F.Cu at (72.2, 187.2)
- added REF**: MountingHole_5mm_Pad, Mounting_Holes:MountingHole_5mm_Pad, F.Cu at (122.7, 187.2)
- added REF**: MountingHole_5mm_Pad, Mounting_Holes:MountingHole_5mm_Pad, F.Cu at (122.7, 22.2)
- added REF**: MountingHole_5mm_Pad, Mounting_Holes:MountingHole_5mm_Pad, F.Cu at (72.2, 22.2)
- moved C2 282.1 mm to (-133.8, -61.6)
- moved C3 282.1 mm to (-133.7, -47.2)
- moved C4 282.1 mm to (-151.6, -33.8)
- moved R25 282.1 mm to (-139.3, -16.6)
- moved R35 282.1 mm to (-173.4, -20.6)
- moved R36 282.1 mm to (-152.6, -36.8)
- moved R37 282.1 mm to (-152.6, -39.8)
- moved R38 282.1 mm to (-152.6, -42.5)
- moved R39 282.1 mm to (-167.2, -20.5)
- moved R40 282.1 mm to (-160.8, -35.5)
- moved R41 282.1 mm to (-160.8, -39.0)
- moved R42 282.1 mm to (-160.8, -42.5)
- moved R43 282.1 mm to (-160.6, -48.0)
- moved R44 282.1 mm to (-154.1, -48.0)
- moved R45 282.1 mm to (-160.8, -50.6)
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Connections:
- A1 pad 1: (no net) -> Net-(A1-Pad1)
- A1 pad 17: (no net) -> Net-(A1-Pad17)
- A1 pad 18: (no net) -> Net-(A1-Pad18)
- A1 pad 2: (no net) -> Net-(A1-Pad2)
- A1 pad 23: (no net) -> Net-(A1-Pad23)
- A1 pad 24: (no net) -> Net-(A1-Pad24)
- A1 pad 25: (no net) -> Net-(A1-Pad25)
- A1 pad 26: (no net) -> Net-(A1-Pad26)
- A1 pad 28: (no net) -> Net-(A1-Pad28)
- A1 pad 3: (no net) -> Net-(A1-Pad3)
- A1 pad 30: (no net) -> Net-(A1-Pad30)
- D1 pad 2: (no net) -> Net-(D1-Pad2)
- J1 pad 2: (no net) -> Net-(J1-Pad2)
- J2 pad 7: (no net) -> Net-(J2-Pad7)
- J3 pad 7: (no net) -> Net-(J3-Pad7)
- J5 pad 2: (no net) -> Net-(J5-Pad2)
- Q10 pad 3: /SUP_GND -> GND
- Q11 pad 3: /SUP_GND -> GND
- Q12 pad 3: /SUP_GND -> GND
- Q13 pad 3: /SUP_GND -> GND
- Q14 pad 3: /SUP_GND -> GND
- Q15 pad 3: /SUP_GND -> GND
- Q16 pad 3: /SUP_GND -> GND
- Q17 pad 3: /SUP_GND -> GND
- Q18 pad 3: /SUP_GND -> GND
- Q9 pad 3: /SUP_GND -> GND
- R27 pad 1: /SUP_GND -> GND
- R28 pad 1: /SUP_GND -> GND
- R29 pad 1: /SUP_GND -> GND
- R30 pad 1: /SUP_GND -> GND
- R31 pad 1: /SUP_GND -> GND
- R32 pad 1: /SUP_GND -> GND
- R33 pad 1: /SUP_GND -> GND
- R34 pad 1: /SUP_GND -> GND
- R44 pad 1: /SUP_GND -> GND
- R46 pad 1: /SUP_GND -> GND
- R48 pad 1: /SUP_GND -> GND
- R50 pad 1: /SUP_GND -> GND
- R52 pad 1: /SUP_GND -> GND
- R54 pad 1: /SUP_GND -> GND
- R56 pad 1: /SUP_GND -> GND
- R58 pad 1: /SUP_GND -> GND
- R67 pad 1: /SUP_GND -> GND
- R69 pad 1: /SUP_GND -> GND
- U1 pad 7: (no net) -> Net-(U1-Pad7)
- U2 pad 10: (no net) -> Net-(U2-Pad10)
- U2 pad 7: (no net) -> Net-(U2-Pad7)
- U6 pad 9: (no net) -> Net-(U6-Pad9)
Routing:
- net /SUP_GND: track 295.7 -> 0.00 mm, vias 1 -> 0
- net GND: track 373.5 -> 102.5 mm, vias 1 -> 0
- net /18V: track 284.6 -> 79.2 mm, vias 1 -> 0
- net /5V: track 180.3 -> 0.00 mm, vias 5 -> 0
- net Net-(A1-Pad20): track 124.0 -> 0.00 mm, vias 6 -> 0
- net /OUT_CLK: track 116.1 -> 0.00 mm, vias 3 -> 0
- net /OUT_LOAD: track 103.5 -> 0.00 mm, vias 4 -> 0
- net /IN_CLK: track 88.1 -> 0.00 mm, vias 3 -> 0
- net /IN_DATA: track 65.8 -> 0.00 mm, vias 1 -> 0
- net /IN_LOAD: track 62.4 -> 0.00 mm, vias 2 -> 0
- net /CO4: track 61.1 -> 0.00 mm
- net /OUT_DATA: track 60.3 -> 0.00 mm, vias 1 -> 0
- net /CI3: track 60.2 -> 0.00 mm, vias 4 -> 0
- net /J12_RO6: track 75.0 -> 15.1 mm
- net /J12_RO2: track 71.7 -> 15.3 mm
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Other:
- board size 128.7 x 81 mm -> 314.6 x 206.8 mm
- net class Default removed
- net class Fett removed
- board text removed: "(c) 2021 bitfield labs"
- board text removed: "+ 18V -"
- board text removed: "1"
- board text removed: "4"
- board text removed: "J133 OUT"
- board text removed: "J134 OUT"
- board text removed: "J135 IN"
- board text removed: "J135 OUT"
- board text removed: "J136 OUT"
- board text removed: "J137 OUT"
- board text removed: "J138 IN"
- board text removed: "J138 OUT"
- board text removed: "v1.5"

Commit message: Layout experiments
Parts:
- moved R45 319.9 mm to (115.4, 110.8)
- moved C4 218.7 mm to (17.4, 105.2)
- moved D1 218.7 mm to (-49.1, 167.4)
- moved R25 218.7 mm to (29.6, 122.4)
- moved R36 218.7 mm to (16.4, 102.2)
- moved R37 218.7 mm to (16.4, 99.2)
- moved R38 218.7 mm to (16.4, 96.5)
- moved R40 218.7 mm to (8.10, 103.5)
- moved R41 218.7 mm to (8.10, 100.0)
- moved R42 218.7 mm to (8.10, 96.5)
- moved R43 218.7 mm to (8.35, 91.0)
- moved R44 218.7 mm to (14.8, 91.0)
- moved R46 218.7 mm to (14.8, 88.3)
- moved R47 218.7 mm to (8.10, 83.0)
- moved R48 218.7 mm to (14.8, 82.9)
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Routing:
- net GND: track 102.5 -> 0.00 mm
- net /18V: track 79.2 -> 0.00 mm
- net /J13_CO8: track 30.9 -> 0.00 mm
- net /J13_CO6: track 29.2 -> 0.00 mm
- net /J12_RO9: track 28.2 -> 0.00 mm
- net /J13_CO2: track 27.5 -> 0.00 mm
- net /J12_RO1: track 27.5 -> 0.00 mm
- net /J13_CO4: track 27.2 -> 0.00 mm
- net /J12_RO5: track 26.3 -> 0.00 mm
- net /J12_RO7: track 26.0 -> 0.00 mm
- net /J12_RO3: track 25.8 -> 0.00 mm
- net /J12_RO10: track 20.0 -> 0.00 mm
- net /J13_CO7: track 18.6 -> 0.00 mm
- net /J13_CO5: track 16.9 -> 0.00 mm
- net /J12_RO8: track 15.4 -> 0.00 mm
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Other:
- board size 314.6 x 206.8 mm -> 81 x 181.4 mm

Commit message: Some progress
Parts:
- moved R67 184.0 mm to (127.2, 95.9), turned to 180 degrees
- moved R26 173.6 mm to (117.2, 95.9)
- moved D1 138.6 mm to (75.9, 107.6)
- moved R52 123.9 mm to (127.2, 108.9), turned to 180 degrees
- moved R54 123.5 mm to (127.2, 112.2), turned to 180 degrees
- moved R56 121.1 mm to (127.2, 99.2), turned to 180 degrees
- moved R46 118.3 mm to (127.2, 125.2)
- moved R53 117.5 mm to (117.2, 112.2)
- moved R50 117.2 mm to (127.2, 118.7)
- moved R48 117.0 mm to (127.2, 115.4)
- moved R44 116.6 mm to (127.2, 121.9)
- moved R55 114.7 mm to (117.2, 99.2)
- moved R49 113.9 mm to (117.2, 118.7)
- moved R47 113.8 mm to (117.2, 115.4)
- moved R43 113.1 mm to (117.2, 121.9)
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Routing:
- net /18V: track 0.00 -> 407.9 mm
- net GND: track 0.00 -> 304.0 mm
- net Net-(Q10-Pad1): track 0.00 -> 94.3 mm
- net /CO8: track 0.00 -> 85.9 mm
- net /CO6: track 0.00 -> 75.9 mm
- net /CO7: track 0.00 -> 75.6 mm
- net /CO5: track 0.00 -> 66.0 mm
- net /CO4: track 0.00 -> 65.2 mm, vias 0 -> 2
- net Net-(Q9-Pad1): track 0.00 -> 65.2 mm
- net Net-(Q11-Pad1): track 0.00 -> 57.0 mm
- net /RO1: track 0.00 -> 54.2 mm, vias 0 -> 2
- net /CO2: track 0.00 -> 52.3 mm, vias 0 -> 2
- net /CO3: track 0.00 -> 51.7 mm, vias 0 -> 2
- net /RO2: track 0.00 -> 51.4 mm, vias 0 -> 2
- net /RO1O: track 0.00 -> 51.2 mm, vias 0 -> 2
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
Commit message: More progress
Parts:
- added C5: 0.33, Capacitor_SMD:C_0805_2012Metric_Pad1.18x1.45mm_HandSolder, F.Cu at (86.6, 63.8)
- C2, C3, C4: footprint Capacitors_SMD:C_0805_HandSoldering -> Capacitor_SMD:C_0805_2012Metric_Pad1.18x1.45mm_HandSolder
- moved C3 96.6 mm to (113.4, 35.0)
- moved C2 87.5 mm to (113.3, 38.4)
- moved R25 65.8 mm to (87.0, 106.3)
- moved SW1 10.8 mm to (72.0, 72.6), turned to -90 degrees
- moved D1 2.60 mm to (78.4, 108.3)
- moved U3 0.40 mm to (79.2, 32.2)
Connections:
- A1 pad 1: Net-(A1-Pad1) -> unconnected-(A1-Pad1)
- A1 pad 17: Net-(A1-Pad17) -> unconnected-(A1-Pad17)
- A1 pad 18: Net-(A1-Pad18) -> unconnected-(A1-Pad18)
- A1 pad 2: Net-(A1-Pad2) -> unconnected-(A1-Pad2)
- A1 pad 23: Net-(A1-Pad23) -> unconnected-(A1-Pad23)
- A1 pad 24: Net-(A1-Pad24) -> unconnected-(A1-Pad24)
- A1 pad 25: Net-(A1-Pad25) -> unconnected-(A1-Pad25)
- A1 pad 26: Net-(A1-Pad26) -> unconnected-(A1-Pad26)
- A1 pad 28: Net-(A1-Pad28) -> unconnected-(A1-Pad28)
- A1 pad 3: Net-(A1-Pad3) -> unconnected-(A1-Pad3)
- A1 pad 30: Net-(A1-Pad30) -> unconnected-(A1-Pad30)
- D1 pad 2: Net-(D1-Pad2) -> unconnected-(D1-Pad2)
- J1 pad 2: Net-(J1-Pad2) -> unconnected-(J1-Pad2)
- J2 pad 7: Net-(J2-Pad7) -> unconnected-(J2-Pad7)
- J3 pad 7: Net-(J3-Pad7) -> unconnected-(J3-Pad7)
- J5 pad 2: Net-(J5-Pad2) -> unconnected-(J5-Pad2)
- U1 pad 7: Net-(U1-Pad7) -> unconnected-(U1-Pad7)
- U2 pad 10: Net-(U2-Pad10) -> unconnected-(U2-Pad10)
- U2 pad 7: Net-(U2-Pad7) -> unconnected-(U2-Pad7)
- U6 pad 9: Net-(U6-Pad9) -> unconnected-(U6-Pad9)
Routing:
- net /18V_IN: track 0.00 -> 209.9 mm
- net GND: track 304.0 -> 465.2 mm, vias 0 -> 3
- net Net-(A1-Pad20): track 0.00 -> 97.6 mm, vias 0 -> 2
- net /18V: track 407.9 -> 480.4 mm
- net /5V: track 0.00 -> 61.4 mm
- net /OUT_CLK: track 0.00 -> 48.0 mm
- net /OUT_LOAD: track 0.00 -> 47.5 mm, vias 0 -> 2
- net /OUT_DATA: track 0.00 -> 41.8 mm, vias 0 -> 1
- net Net-(U5-Pad9): track 0.00 -> 38.4 mm
- net Net-(U5-Pad15): track 0.00 -> 16.0 mm, vias 0 -> 2
- net Net-(A1-Pad19): track 0.00 -> 9.63 mm
- net Net-(A1-Pad14): track 0.00 -> 6.77 mm
- net Net-(A1-Pad12): track 0.00 -> 6.77 mm
- net Net-(A1-Pad11): track 0.00 -> 6.77 mm
- net Net-(A1-Pad13): track 0.00 -> 6.77 mm
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
Commit message: hui
Parts:
- moved R24 38.6 mm to (82.1, 66.3), turned to 180 degrees
- moved R23 34.8 mm to (82.1, 63.4), turned to 180 degrees
- moved R22 30.9 mm to (82.1, 60.5), turned to 180 degrees
- moved R21 27.1 mm to (82.1, 57.6), turned to 180 degrees
- moved R8 26.9 mm to (92.6, 66.3), turned to 0 degrees
- moved D6 23.9 mm to (102.7, 57.6), turned to 0 degrees
- moved D2 23.5 mm to (102.7, 46.0), turned to 0 degrees
- moved R20 23.5 mm to (82.1, 54.7), turned to 180 degrees
- moved R7 23.1 mm to (92.5, 63.4), turned to 0 degrees
- moved D7 22.1 mm to (102.7, 60.5), turned to 0 degrees
- moved D8 20.7 mm to (102.7, 63.4), turned to 0 degrees
- moved D3 20.7 mm to (102.7, 49.0), turned to 0 degrees
- moved R19 20.1 mm to (82.1, 51.8), turned to 180 degrees
- moved D9 20.0 mm to (102.7, 66.3), turned to 0 degrees
- moved R16 19.4 mm to (112.8, 46.1), turned to 180 degrees
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
Commit message: hmmm
Parts:
- renumbered REF** to HOLE1, REF** to HOLE2, REF** to HOLE3, REF** to HOLE4
Routing:
- net GND: track 465.2 -> 534.1 mm, vias 3 -> 11
- net /CI7: track 0.00 -> 44.6 mm
- net /CI8: track 0.00 -> 42.7 mm
- net /5V: track 61.4 -> 81.6 mm
- net Net-(J1-Pad1): track 0.00 -> 19.5 mm
- net /CI6: track 0.00 -> 19.2 mm
- net /CI3: track 0.00 -> 19.2 mm
- net /CI2: track 0.00 -> 19.2 mm
- net /CI4: track 0.00 -> 19.2 mm
- net /CI5: track 0.00 -> 19.2 mm
- net /CI1: track 0.00 -> 19.2 mm
- net /RI1: track 0.00 -> 17.1 mm
- net Net-(J1-Pad3): track 0.00 -> 17.0 mm
- net /RI2: track 0.00 -> 16.7 mm
- net Net-(J1-Pad4): track 0.00 -> 16.5 mm
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
Commit message: hmmm
Parts:
- moved C3 5.80 mm to (110.8, 34.9)
- moved C2 4.96 mm to (110.8, 28.1)
- moved U2 3.73 mm to (107.2, 73.0)
- moved C5 2.51 mm to (96.1, 73.1)
Routing:
- net /5V: track 81.6 -> 354.9 mm, vias 0 -> 1
- net GND: track 534.1 -> 724.0 mm, vias 11 -> 14
- net /RI10: track 0.00 -> 110.6 mm
- net /RI9: track 0.00 -> 89.6 mm
- net /RI8: track 14.3 -> 75.7 mm, vias 0 -> 1
- net /RI7: track 13.8 -> 70.3 mm, vias 0 -> 1
- net /RI6: track 14.9 -> 63.0 mm, vias 0 -> 1
- net /IN_CLK: track 0.00 -> 43.9 mm
- net /OUT_LOAD: track 47.5 -> 90.1 mm
- net /IN_LOAD: track 0.00 -> 41.0 mm
- net /OUT_CLK: track 48.0 -> 88.7 mm
- net /RI5: track 15.4 -> 49.9 mm, vias 0 -> 1
- net /18V: track 480.4 -> 511.9 mm
- net /RI4: track 15.8 -> 42.0 mm, vias 0 -> 1
- net /RI3: track 16.3 -> 42.3 mm, vias 0 -> 1
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
Commit message: hmmm
Routing:
- net Net-(U1-Pad10): track 0.00 -> 27.3 mm, vias 0 -> 2
- net /RI5: track 49.9 -> 64.3 mm
- net /RI8: track 75.7 -> 79.7 mm
- net /RI6: track 63.0 -> 66.9 mm
- net /RI7: track 70.3 -> 73.9 mm
Changed lines of the file:
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@@
   (segment (start 109.8872 63.6128) (end 106.4 67.1) (width 0.5) (layer "B.Cu") (net 6))
   (segment (start 127.5 63.6128) (end 109.8872 63.6128) (width 0.5) (layer "B.Cu") (net 6))
-  (segment (start 105.295 73.695) (end 105.295 73.194011) (width 0.5) (layer "F.Cu") (net 7))
+  (segment (start 106.288166 72.701834) (end 115.172516 72.701834) (width 0.5) (layer "F.Cu") (net 7))
   (segment (start 119.0954 59.6504) (end 114.175 54.73) (width 0.5) (layer "F.Cu") (net 7))
   (segment (start 105.295 73.695) (end 105.295 75.7) (width 0.5) (layer "F.Cu") (net 7))
+  (segment (start 105.295 73.695) (end 106.288166 72.701834) (width 0.5) (layer "F.Cu") (net 7))
   (segment (start 127.5 59.6504) (end 119.0954 59.6504) (width 0.5) (layer "F.Cu") (net 7))
-  (segment (start 105.295 73.194011) (end 104.7 72.599011) (width 0.5) (layer "F.Cu") (net 7))
-  (via (at 104.7 72.599011) (size 0.6) (drill 0.4) (layers "F.Cu" "B.Cu") (net 7))
-  (segment (start 104.5 67.86932) (end 104.5 72.399011) (width 0.5) (layer "B.Cu") (net 7))
-  (segment (start 104.5 72.399011) (end 104.7 72.599011) (width 0.5) (layer "B.Cu") (net 7))
-  (segment (start 127.5 59.6504) (end 112.71892 59.6504) (width 0.5) (layer "B.Cu") (net 7))
-  (segment (start 112.71892 59.6504) (end 104.5 67.86932) (width 0.5) (layer "B.Cu") (net 7))
+  (segment (start 115.172516 72.701834) (end 120.310351 77.839669) (width 0.5) (layer "F.Cu") (net 7))
+  (via (at 120.310351 77.839669) (size 0.6) (drill 0.4) (layers "F.Cu" "B.Cu") (net 7))
+  (segment (start 128 59.6504) (end 130.22692 61.87732) (width 0.5) (layer "B.Cu") (net 7))
+  (segment (start 130.22692 77.47308) (end 129.8 77.9) (width 0.5) (layer "B.Cu") (net 7))
+  (segment (start 129.8 77.9) (end 120.3 77.9) (width 0.5) (layer "B.Cu") (net 7))
+  (segment (start 130.22692 61.87732) (end 130.22692 77.47308) (width 0.5) (layer "B.Cu") (net 7))
+  (segment (start 127.5 59.6504) (end 128 59.6504) (width 0.5) (layer "B.Cu") (net 7))
   (segment (start 118.023 55.688) (end 114.175 51.84) (width 0.5) (layer "F.Cu") (net 8))
   (segment (start 106.565 77.465) (end 106.6 77.5) (width 0.5) (layer "F.Cu") (net 8))
@@
   (segment (start 127.5 55.688) (end 118.023 55.688) (width 0.5) (layer "F.Cu") (net 8))
   (via (at 106.6 77.5) (size 0.6) (drill 0.4) (layers "F.Cu" "B.Cu") (net 8))
-  (segment (start 129.999022 77.5) (end 107.7 77.5) (width 0.5) (layer "B.Cu") (net 8))
-  (segment (start 129.99952 77.499502) (end 129.999022 77.5) (width 0.5) (layer "B.Cu") (net 8))
-  (segment (start 129.99952 58.18752) (end 129.99952 77.499502) (width 0.5) (layer "B.Cu") (net 8))
-  (segment (start 107.7 77.5) (end 106.6 77.5) (width 0.5) (layer "B.Cu") (net 8))
-  (segment (start 127.5 55.688) (end 129.99952 58.18752) (width 0.5) (layer "B.Cu") (net 8))
+  (segment (start 130.110461 78.64952) (end 119.989538 78.64952) (width 0.5) (layer "B.Cu") (net 8))
+  (segment (start 118.840018 77.5) (end 106.6 77.5) (width 0.5) (layer "B.Cu") (net 8))
+  (segment (start 130.97644 56.66444) (end 130.97644 77.783542) (width 0.5) (layer "B.Cu") (net 8))
+  (segment (start 119.989538 78.64952) (end 118.840018 77.5) (width 0.5) (layer "B.Cu") (net 8))
+  (segment (start 130.97644 77.783542) (end 130.110461 78.64952) (width 0.5) (layer "B.Cu") (net 8))
+  (segment (start 127.5 55.688) (end 130 55.688) (width 0.5) (layer "B.Cu") (net 8))
+  (segment (start 130 55.688) (end 130.97644 56.66444) (width 0.5) (layer "B.Cu") (net 8))
   (segment (start 115.3618 47.7632) (end 114.175 48.95) (width 0.5) (layer "F.Cu") (net 9))
   (segment (start 107.835 76.835) (end 109.1 78.1) (width 0.5) (layer "F.Cu") (net 9))
@@
   (segment (start 117.8 78.1) (end 118.3 78.6) (width 0.5) (layer "F.Cu") (net 9))
   (via (at 118.3 78.6) (size 0.6) (drill 0.4) (layers "F.Cu" "B.Cu") (net 9))
-  (segment (start 130.74904 51.01224) (end 130.74904 77.85096) (width 0.5) (layer "B.Cu") (net 9))
-  (segment (start 127.5 47.7632) (end 130.74904 51.01224) (width 0.5) (layer "B.Cu") (net 9))
-  (segment (start 130 78.6) (end 118.3 78.6) (width 0.5) (layer "B.Cu") (net 9))
-  (segment (start 130.74904 77.85096) (end 130 78.6) (width 0.5) (layer "B.Cu") (net 9))
-  (segment (start 120.3 79.46932) (end 120.3 79.6) (width 0.5) (layer "F.Cu") (net 10))
+  (segment (start 119.099039 79.399039) (end 118.3 78.6) (width 0.5) (layer "B.Cu") (net 9))
+  (segment (start 127.5 47.7632) (end 129.8632 47.7632) (width 0.5) (layer "B.Cu") (net 9))
+  (segment (start 130.420924 79.399039) (end 119.099039 79.399039) (width 0.5) (layer "B.Cu") (net 9))
+  (segment (start 131.725959 78.094004) (end 130.420924 79.399039) (width 0.5) (layer "B.Cu") (net 9))
+  (segment (start 131.72596 49.62596) (end 131.725959 78.094004) (width 0.5) (layer "B.Cu") (net 9))
+  (segment (start 129.8632 47.7632) (end 131.72596 49.62596) (width 0.5) (layer "B.Cu") (net 9))
+  (segment (start 120.5 80.198539) (end 120.5 79.66932) (width 0.5) (layer "F.Cu") (net 10))
   (segment (start 109.105 76.95) (end 109.455 77.3) (width 0.5) (layer "F.Cu") (net 10))
   (segment (start 109.105 75.7) (end 109.105 76.95) (width 0.5) (layer "F.Cu") (net 10))
   (segment (start 116.4342 43.8008) (end 114.175 46.06) (width 0.5) (layer "F.Cu") (net 10))
-  (segment (start 118.13068 77.3) (end 120.3 79.46932) (width 0.5) (layer "F.Cu") (net 10))
+  (segment (start 120.5 79.66932) (end 118.13068 77.3) (width 0.5) (layer "F.Cu") (net 10))
   (segment (start 109.455 77.3) (end 118.13068 77.3) (width 0.5) (layer "F.Cu") (net 10))
   (segment (start 127.5 43.8008) (end 116.4342 43.8008) (width 0.5) (layer "F.Cu") (net 10))
-  (via (at 120.3 79.6) (size 0.6) (drill 0.4) (layers "F.Cu" "B.Cu") (net 10))
-  (segment (start 131.49856 78.161422) (end 130.059982 79.6) (width 0.5) (layer "B.Cu") (net 10))
-  (segment (start 131.49856 47.79936) (end 131.49856 78.161422) (width 0.5) (layer "B.Cu") (net 10))
-  (segment (start 127.5 43.8008) (end 131.49856 47.79936) (width 0.5) (layer "B.Cu") (net 10))
-  (segment (start 130.059982 79.6) (end 120.3 79.6) (width 0.5) (layer "B.Cu") (net 10))
+  (via (at 120.5 80.198539) (size 0.6) (drill 0.4) (layers "F.Cu" "B.Cu") (net 10))
+  (segment (start 132.47548 78.404464) (end 130.731385 80.148559) (width 0.5) (layer "B.Cu") (net 10))
+  (segment (start 132.47548 77.22452) (end 132.47548 78.404464) (width 0.5) (layer "B.Cu") (net 10))
+  (segment (start 132.47548 77.22452) (end 132.47548 45.8) (width 0.5) (layer "B.Cu") (net 10))
+  (segment (start 130.47628 43.8008) (end 127.5 43.8008) (width 0.5) (layer "B.Cu") (net 10))
+  (segment (start 120.54998 80.148559) (end 120.5 80.198539) (width 0.5) (layer "B.Cu") (net 10))
+  (segment (start 130.731385 80.148559) (end 120.54998 80.148559) (width 0.5) (layer "B.Cu") (net 10))
+  (segment (start 132.47548 45.8) (end 130.47628 43.8008) (width 0.5) (layer "B.Cu") (net 10))
   (segment (start 112.95 84.625) (end 113.025 84.7) (width 0.5) (layer "F.Cu") (net 11))
   (segment (start 124.027152 121.927152) (end 122.4 120.3) (width 0.5) (layer "F.Cu") (net 11))
@@
   (segment (start 103.6 79.8) (end 101.1 77.3) (width 0.5) (layer "F.Cu") (net 37))
   (segment (start 103.675 74.1) (end 104.025 74.45) (width 0.5) (layer "F.Cu") (net 37))
+  (segment (start 111.645 70.3) (end 111.645 69.045) (width 0.5) (layer "F.Cu") (net 38))
+  (segment (start 99.7 70.4) (end 88.970978 70.4) (width 0.5) (layer "F.Cu") (net 38))
+  (segment (start 88.970978 70.4) (end 87.925 71.445978) (width 0.5) (layer "F.Cu") (net 38))
+  (segment (start 111.645 69.045) (end 111 68.4) (width 0.5) (layer "F.Cu") (net 38))
+  (segment (start 87.925 71.445978) (end 87.925 72.225) (width 0.5) (layer "F.Cu") (net 38))
+  (via (at 99.7 70.4) (size 0.6) (drill 0.4) (layers "F.Cu" "B.Cu") (net 38))
+  (via (at 111 68.4) (size 0.6) (drill 0.4) (layers "F.Cu" "B.Cu") (net 38))
+  (segment (start 111 68.4) (end 101.7 68.4) (width 0.5) (layer "B.Cu") (net 38))
+  (segment (start 101.7 68.4) (end 99.7 70.4) (width 0.5) (layer "B.Cu") (net 38))
   (segment (start 97.1 92.55) (end 103.75 99.2) (width 0.5) (layer "F.Cu") (net 39))
   (segment (start 95.4 91.5) (end 96.1 91.5) (width 0.5) (layer "F.Cu") (net 39))
