File: afterglow_stern_pcb_v10/afterglow_nano_smd.kicad_pcb (KiCad board)
At the start: 2 copper layers, 81 x 181.4 mm, 123 parts, among them J1 J13_IN_C, J2 J12_IN_R, J3 J12_OUT_R, J5 J13_OUT_C, Q1 FQP11P06, Q10 FQP13N06L, Q11 FQP13N06L, Q12 FQP13N06L, Q13 FQP13N06L, Q14 FQP13N06L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

Commit message: Juhu
Routing:
- net /CI1: track 19.2 -> 47.6 mm, vias 0 -> 2
- net /CI5: track 19.2 -> 44.7 mm, vias 0 -> 2
- net /CI2: track 19.2 -> 44.3 mm, vias 0 -> 2
- net /CI6: track 19.2 -> 42.0 mm, vias 0 -> 2
- net /CI3: track 19.2 -> 41.6 mm, vias 0 -> 2
- net /CI7: track 19.2 -> 38.8 mm, vias 0 -> 2
- net /18V: track 511.9 -> 531.1 mm, vias 0 -> 1
- net /CI4: track 19.7 -> 38.8 mm, vias 0 -> 2
- net /CI8: track 19.2 -> 36.1 mm, vias 0 -> 2
- net GND: track 724.0 -> 728.4 mm
- net /RO9: track 50.3 -> 52.2 mm

Commit message: Juhu
Connections:
- HOLE1 pad 1: (no net) -> GND
- HOLE2 pad 1: (no net) -> GND
- HOLE3 pad 1: (no net) -> GND
- HOLE4 pad 1: (no net) -> GND
Routing:
- added copper zone on B.Cu, net GND
Changed lines of the file:
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@@
     (fp_circle (center 0 0) (end 5 0) (layer "Cmts.User") (width 0.15) (fill none))
     (fp_circle (center 0 0) (end 5.25 0) (layer "F.CrtYd") (width 0.05) (fill none))
-    (pad "1" thru_hole circle locked (at 0 0) (size 10 10) (drill 5) (layers *.Cu *.Mask))
+    (pad "1" thru_hole circle locked (at 0 0) (size 10 10) (drill 5) (layers *.Cu *.Mask)
+      (net 2 "GND"))
   )
   (footprint "Mounting_Holes:MountingHole_5mm_Pad" (layer "F.Cu")
@@
     (fp_circle (center 0 0) (end 5 0) (layer "Cmts.User") (width 0.15) (fill none))
     (fp_circle (center 0 0) (end 5.25 0) (layer "F.CrtYd") (width 0.05) (fill none))
-    (pad "1" thru_hole circle locked (at 0 0) (size 10 10) (drill 5) (layers *.Cu *.Mask))
+    (pad "1" thru_hole circle locked (at 0 0) (size 10 10) (drill 5) (layers *.Cu *.Mask)
+      (net 2 "GND"))
   )
   (footprint "Mounting_Holes:MountingHole_5mm_Pad" (layer "F.Cu")
@@
     (fp_circle (center 0 0) (end 5 0) (layer "Cmts.User") (width 0.15) (fill none))
     (fp_circle (center 0 0) (end 5.25 0) (layer "F.CrtYd") (width 0.05) (fill none))
-    (pad "1" thru_hole circle locked (at 0 0) (size 10 10) (drill 5) (layers *.Cu *.Mask))
+    (pad "1" thru_hole circle locked (at 0 0) (size 10 10) (drill 5) (layers *.Cu *.Mask)
+      (net 2 "GND"))
   )
   (footprint "Mounting_Holes:MountingHole_5mm_Pad" (layer "F.Cu")
@@
     (fp_circle (center 0 0) (end 5 0) (layer "Cmts.User") (width 0.15) (fill none))
     (fp_circle (center 0 0) (end 5.25 0) (layer "F.CrtYd") (width 0.05) (fill none))
-    (pad "1" thru_hole circle locked (at 0 0) (size 10 10) (drill 5) (layers *.Cu *.Mask))
+    (pad "1" thru_hole circle locked (at 0 0) (size 10 10) (drill 5) (layers *.Cu *.Mask)
+      (net 2 "GND"))
   )
   (footprint "Capacitors_THT:CP_Radial_D16.0mm_P7.50mm" (layer "F.Cu")
@@
   (segment (start 107.191716 126.536716) (end 107.191716 114.282351) (width 0.5) (layer "F.Cu") (net 98))
   (segment (start 109.295 128.64) (end 107.191716 126.536716) (width 0.5) (layer "F.Cu") (net 98))
+  (zone (net 2) (net_name "GND") (layer "B.Cu") (name "GND") (hatch edge 0.508)
+    (connect_pads (clearance 0.508))
+    (min_thickness 0.254) (filled_areas_thickness no)
+    (fill yes (thermal_gap 0.508) (thermal_bridge_width 0.508) (smoothing fillet))
+    (polygon
+      (pts
+        (xy 136 18.1)
+        (xy 135.9 190)
+        (xy 133 193)
+        (xy 61 193)
+        (xy 59.1 190)
+        (xy 58.9 18.1)
+        (xy 61 16)
+        (xy 134 16)
+      )
+    )
+  )
   (group "" locked (id 503a3d5c-692f-44ea-91f8-862b78ede738)
     (members
