File: afterglow_pcb_v15/afterglow_nano_smd.kicad_sch (KiCad schematic)
At the start: 125 parts, among them J1 J137_IN_C, J2 J133_IN_R, J3 Conn_Power, J4 J133_OUT_R, J5 J137_OUT_C, J6 J134_OUT_R, J7 J138_OUT_C, J8 J135_OUT_R, J9 136_OUT_C, Q1 FQP11P06, Q10 FQP13N06L, Q11 FQP13N06L, Q12 FQP13N06L, Q13 FQP13N06L, Q14 FQP13N06L, Q15 FQP13N06L, Q16 FQP13N06L, Q2 FQP11P06, Q3 FQP11P06, Q4 FQP11P06, Q5 FQP11P06, Q6 FQP11P06, Q7 FQP11P06, Q8 FQP11P06, Q9 FQP13N06L, SW1 CFG, U1 74LS165, U2 74LS165, U3 5V_Regulator, U5 74HC595, U6 74HC595, U7 ULN2803A

Commit message: Added JLCPCB production files
Parts:
- C1: JLCPCB (none) -> C10750
- C2, C4: JLCPCB (none) -> C1740
- C3: JLCPCB (none) -> C49678
- D1, D10, D11, D12, D13, D14, D15, D16, D17: JLCPCB (none) -> C50603
- D2, D3, D4, D5, D6, D7, D8, D9: JLCPCB (none) -> C124651
- F1: JLCPCB (none) -> C3130
- J1, J5, J7: JLCPCB (none) -> C239400
- J2, J4, J6, J8: JLCPCB (none) -> C509152
- J3: JLCPCB (none) -> C239393
- J9: JLCPCB (none) -> C10585
- Q1, Q2, Q3, Q4, Q5, Q6, Q7, Q8: JLCPCB (none) -> C693361
- Q10, Q11, Q12, Q13, Q14, Q15, Q16, Q9: JLCPCB (none) -> C243082
- R1, R10, R11, R12, R13, R14, R15, R16, R17, R18, R19, R2, R20, R21, R22, R23, R24, R3, R4, R5, R6, R7, R8, R9: JLCPCB (none) -> C17513
- R25, R27, R28, R29, R30, R31, R32, R33, R34, R44, R46, R48, R50, R52, R54, R56, R58, R59, R60, R61, R62, R63, R64, R65, R66: JLCPCB (none) -> C17414
- R26: JLCPCB (none) -> C68608
- R35, R36, R37, R38, R39, R40, R41, R42: JLCPCB (none) -> C17604
- R43, R45, R47, R49, R51, R53, R55, R57: JLCPCB (none) -> C17557
- R67: JLCPCB (none) -> C17477
- SW1: JLCPCB (none) -> C559139
- U1, U2: JLCPCB (none) -> C5613
- U3: JLCPCB (none) -> C111887
- U5, U6: JLCPCB (none) -> C5947
- U7: JLCPCB (none) -> C9683
