File: afterglow_pcb_v30/hat_modder/hat_modder.kicad_sch (KiCad schematic)
At the start: 28 parts, among them J1 Conn_01x10_Pin, J2 Conn_02x03_Odd_Even, J3 Conn_02x03_Odd_Even, J4 Conn_01x10_Pin, J5 Conn_01x02_Socket, J6 Conn_01x02_Socket, J7 Conn_01x02_Socket, J8 Conn_01x02_Socket, U1 74HC244, U2 74HC595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

Commit message: hat progress
Parts:
- renumbered ST_LED1 to D1, ST_LED2 to D2, ST_LED3 to D3, ST_LED4 to D4
Connections:
- net RI1 is gone; now on net GND: U3.2, U4.2, U5.2, U6.2

Commit message: hat progress
Parts:
- D1, D2, D3, D4: JLCPCB C72038 -> C2296
- R1, R6, R7, R8, R9: JLCPCB C11702 -> C17513
- U1: JLCPCB (none) -> C6835
- U2: JLCPCB (none) -> C5947
Changed lines of the file:
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@@
 			)
 		)
-		(property "JLCPCB" "C72038"
+		(property "JLCPCB" "C2296"
 			(at 239.395 143.51 90)
 			(effects
@@
 			)
 		)
+		(property "JLCPCB" "C6835"
+			(at 134.62 146.05 0)
+			(effects
+				(font
+					(size 1.524 1.524)
+				)
+				(hide yes)
+			)
+		)
 		(pin "8"
 		)
@@
 			)
 		)
-		(property "JLCPCB" "C72038"
+		(property "JLCPCB" "C2296"
 			(at 206.375 143.51 90)
 			(effects
@@
 			)
 		)
+		(property "JLCPCB" "C5947"
+			(at 135.255 84.455 0)
+			(effects
+				(font
+					(size 1.524 1.524)
+				)
+				(hide yes)
+			)
+		)
 		(pin "4"
 		)
@@
 			)
 		)
-		(property "JLCPCB" "C11702"
+		(property "JLCPCB" "C17513"
 			(at 233.045 139.7 90)
 			(effects
@@
 			)
 		)
-		(property "JLCPCB" "C11702"
+		(property "JLCPCB" "C17513"
 			(at 200.025 117.475 90)
 			(effects
@@
 			)
 		)
-		(property "JLCPCB" "C11702"
+		(property "JLCPCB" "C17513"
 			(at 200.025 139.7 90)
 			(effects
@@
 			)
 		)
-		(property "JLCPCB" "C11702"
+		(property "JLCPCB" "C17513"
 			(at 233.045 117.475 90)
 			(effects
@@
 			)
 		)
-		(property "JLCPCB" "C11702"
+		(property "JLCPCB" "C17513"
 			(at 117.475 89.535 90)
 			(effects
@@
 			)
 		)
-		(property "JLCPCB" "C72038"
+		(property "JLCPCB" "C2296"
 			(at 206.375 121.285 90)
 			(effects
@@
 			)
 		)
-		(property "JLCPCB" "C72038"
+		(property "JLCPCB" "C2296"
 			(at 239.395 121.285 90)
 			(effects
